Commit message: upload files

File: factory_amr_description/urdf/factory_amr.xacro (robot description, xacro)
@@ -24,5 +24,8 @@
   </collision>
 </link>
-<link name="right_wheel_1">
+<gazebo reference="base_link">
+  <material>Gazebo/White</material>
+</gazebo>
+<link name="right_wheel">
   <inertial>
     <origin xyz="-1.5713222806367798e-17 -0.03750000000000003 0.0" rpy="0 0 0"/>
@@ -35,5 +38,5 @@
       <mesh filename="file://$(find factory_amr_description)/meshes/right_wheel_1.stl" scale="0.001 0.001 0.001"/>
     </geometry>
-    <material name="silver"/>
+    <material name="black"/>
   </visual>
   <collision>
@@ -44,5 +47,8 @@
   </collision>
 </link>
-<link name="left_wheel_1">
+<gazebo reference="right_wheel">
+  <material>Gazebo/Black</material>
+</gazebo>
+<link name="left_wheel">
   <inertial>
     <origin xyz="0.0 0.03749999999999998 1.3877787807814457e-17" rpy="0 0 0"/>
@@ -55,5 +61,5 @@
       <mesh filename="file://$(find factory_amr_description)/meshes/left_wheel_1.stl" scale="0.001 0.001 0.001"/>
     </geometry>
-    <material name="silver"/>
+    <material name="black"/>
   </visual>
   <collision>
@@ -64,5 +70,8 @@
   </collision>
 </link>
-<link name="revolute_1">
+<gazebo reference="left_wheel">
+  <material>Gazebo/Black</material>
+</gazebo>
+<link name="luggage">
   <inertial>
     <origin xyz="0.2776968707983327 -0.2999999999999999 0.08670656285317513" rpy="0 0 0"/>
@@ -75,5 +84,5 @@
       <mesh filename="file://$(find factory_amr_description)/meshes/revolute_1.stl" scale="0.001 0.001 0.001"/>
     </geometry>
-    <material name="silver"/>
+    <material name="orange"/>
   </visual>
   <collision>
@@ -84,5 +93,8 @@
   </collision>
 </link>
-<link name="lidar_1">
+<gazebo reference="luggage">
+  <material>Gazebo/Orange</material>
+</gazebo>
+<link name="laser_frame">
   <inertial>
     <origin xyz="-7.237528875152536e-18 -1.447505775030507e-17 0.010000000000000009" rpy="0 0 0"/>
@@ -95,5 +107,5 @@
       <mesh filename="file://$(find factory_amr_description)/meshes/lidar_1.stl" scale="0.001 0.001 0.001"/>
     </geometry>
-    <material name="silver"/>
+    <material name="blue"/>
   </visual>
   <collision>
@@ -104,5 +116,5 @@
   </collision>
 </link>
-<link name="imu_1">
+<link name="imu">
   <inertial>
     <origin xyz="0.0 0.0 -0.0050000000000000044" rpy="0 0 0"/>
@@ -115,5 +127,5 @@
       <mesh filename="file://$(find factory_amr_description)/meshes/imu_1.stl" scale="0.001 0.001 0.001"/>
     </geometry>
-    <material name="silver"/>
+    <material name="red"/>
   </visual>
   <collision>
@@ -124,5 +136,8 @@
   </collision>
 </link>
-<link name="camera_1">
+<gazebo reference="imu">
+  <material>Gazebo/Red</material>
+</gazebo>
+<link name="camera">
   <inertial>
     <origin xyz="0.010000000000000064 0.0 0.0" rpy="0 0 0"/>
@@ -135,5 +150,5 @@
       <mesh filename="file://$(find factory_amr_description)/meshes/camera_1.stl" scale="0.001 0.001 0.001"/>
     </geometry>
-    <material name="silver"/>
+    <material name="red"/>
   </visual>
   <collision>
@@ -144,37 +159,95 @@
   </collision>
 </link>
-<joint name="Revolute 7" type="continuous">
+<joint name="right_wheel_joint" type="continuous">
   <origin xyz="0.0 -0.25 0.1" rpy="0 0 0"/>
   <parent link="base_link"/>
-  <child link="right_wheel_1"/>
+  <child link="right_wheel"/>
   <axis xyz="0.0 -1.0 0.0"/>
 </joint>
-<joint name="Revolute 8" type="continuous">
+<joint name="left_wheel_joint" type="continuous">
   <origin xyz="0.0 0.25 0.1" rpy="0 0 0"/>
   <parent link="base_link"/>
-  <child link="left_wheel_1"/>
+  <child link="left_wheel"/>
   <axis xyz="0.0 1.0 0.0"/>
 </joint>
-<joint name="Revolute 9" type="revolute">
+<joint name="luggage_joint" type="revolute">
   <origin xyz="-0.325 0.3 0.525" rpy="0 0 0"/>
   <parent link="base_link"/>
-  <child link="revolute_1"/>
+  <child link="luggage"/>
   <axis xyz="0.0 -1.0 0.0"/>
   <limit upper="0.785398" lower="0.0" effort="100" velocity="100"/>
 </joint>
-<joint name="Rigid 10" type="fixed">
+<joint name="laser_joint" type="fixed">
   <origin xyz="0.0 0.0 0.26" rpy="0 0 0"/>
   <parent link="base_link"/>
-  <child link="lidar_1"/>
-</joint>
-<joint name="Rigid 11" type="fixed">
+  <child link="laser_frame"/>
+</joint>
+<joint name="imu_joint" type="fixed">
   <origin xyz="0.0 0.0 0.23" rpy="0 0 0"/>
   <parent link="base_link"/>
-  <child link="imu_1"/>
-</joint>
-<joint name="Rigid 12" type="fixed">
+  <child link="imu"/>
+</joint>
+<joint name="camera_joint" type="fixed">
   <origin xyz="0.39 0.0 0.475" rpy="0 0 0"/>
   <parent link="base_link"/>
-  <child link="camera_1"/>
-</joint>
+  <child link="camera"/>
+</joint>
+<joint name="camera_optical_joint" type="fixed">
+  <origin xyz="0.0 0.0 0.0" rpy="${-pi/2} 0 ${-pi/2}"/>
+  <parent link="camera"/>
+  <child link="camera_optical"/>
+</joint>
+<link name="camera_optical" type="fixed"></link>
+<gazebo reference="laser_frame">
+  <material>Gazebo/Blue</material>
+  <sensor name="laser" type="ray">
+    <pose> 0 0 0 0 0 0 </pose>
+    <visualize>true</visualize>
+    <update_rate>10</update_rate>
+    <ray>
+      <scan>
+        <horizontal>
+          <samples>360</samples>
+          <resolution>1</resolution>
+          <min_angle>-3.14</min_angle>
+          <max_angle>3.14</max_angle>
+        </horizontal>
+      </scan>
+      <range>
+        <min>0.4</min>
+        <max>12</max>
+      </range>
+    </ray>
+    <plugin name="laser_controller" filename="libgazebo_ros_ray_sensor.so">
+      <ros>
+        <argument>~/out:=scan</argument>
+      </ros>
+      <output_type>sensor_msgs/LaserScan</output_type>
+      <frame_name>laser_frame</frame_name>
+    </plugin>
+  </sensor>
+</gazebo>
+<gazebo reference="camera">
+  <material>Gazebo/Red</material>
+  <sensor name="camera" type="camera">
+    <pose> 0 0 0 0 0 0 </pose>
+    <visualize>true</visualize>
+    <update_rate>10</update_rate>
+    <camera>
+      <horizontal_fov>1.089</horizontal_fov>
+      <image>
+        <format>R8G8B8</format>
+        <width>640</width>
+        <height>480</height>
+      </image>
+      <clip>
+        <near>0.05</near>
+        <far>8.0</far>
+      </clip>
+    </camera>
+    <plugin name="camera_controller" filename="libgazebo_ros_camera.so">
+      <frame_name>camera_optical</frame_name>
+    </plugin>
+  </sensor>
+</gazebo>
 </robot>

File: factory_amr_description/urdf/materials.xacro (robot description, xacro)
@@ -4,3 +4,15 @@
   <color rgba="0.700 0.700 0.700 1.000"/>
 </material>
+<material name="black">
+  <color rgba="0.000 0.000 0.000 1.000"/>
+</material>
+<material name="red">
+  <color rgba="0.800 0.000 0.000 1.000"/>
+</material>
+<material name="blue">
+  <color rgba="0.000 0.000 0.700 1.000"/>
+</material>
+<material name="orange">
+  <color rgba="1.000 0.4235 0.0392 1.000"/>
+</material>
 </robot>

Commit message: Change TF of wheels

File: factory_amr_description/urdf/factory_amr.xacro (robot description, xacro)
@@ -24,12 +24,29 @@
   </collision>
 </link>
-<gazebo reference="base_link">
-  <material>Gazebo/White</material>
-</gazebo>
-<link name="right_wheel">
+<link name="left_wheel_1">
   <inertial>
-    <origin xyz="-1.5713222806367798e-17 -0.03750000000000003 0.0" rpy="0 0 0"/>
-    <mass value="2.1531676424929196"/>
-    <inertia ixx="0.006279" iyy="0.010596" izz="0.006279" ixy="0.0" iyz="-0.0" ixz="-0.0"/>
+    <origin xyz="0.0 0.03749999999999998 0.0" rpy="0 0 0"/>
+    <mass value="18.49612674800992"/>
+    <inertia ixx="0.05491" iyy="0.092481" izz="0.05491" ixy="0.0" iyz="0.0" ixz="0.0"/>
+  </inertial>
+  <visual>
+    <origin xyz="-0.0 -0.25 -0.1" rpy="0 0 0"/>
+    <geometry>
+      <mesh filename="file://$(find factory_amr_description)/meshes/left_wheel_1.stl" scale="0.001 0.001 0.001"/>
+    </geometry>
+    <material name="silver"/>
+  </visual>
+  <collision>
+    <origin xyz="-0.0 -0.25 -0.1" rpy="0 0 0"/>
+    <geometry>
+      <mesh filename="file://$(find factory_amr_description)/meshes/left_wheel_1.stl" scale="0.001 0.001 0.001"/>
+    </geometry>
+  </collision>
+</link>
+<link name="right_wheel_1">
+  <inertial>
+    <origin xyz="1.5440061600325417e-17 -0.03749999999999998 0.0" rpy="0 0 0"/>
+    <mass value="18.496126748009903"/>
+    <inertia ixx="0.05491" iyy="0.092481" izz="0.05491" ixy="-0.0" iyz="0.0" ixz="0.0"/>
   </inertial>
   <visual>
@@ -38,5 +55,5 @@
       <mesh filename="file://$(find factory_amr_description)/meshes/right_wheel_1.stl" scale="0.001 0.001 0.001"/>
     </geometry>
-    <material name="black"/>
+    <material name="silver"/>
   </visual>
   <collision>
@@ -47,45 +64,19 @@
   </collision>
 </link>
-<gazebo reference="right_wheel">
-  <material>Gazebo/Black</material>
-</gazebo>
-<link name="left_wheel">
+<link name="revolute_1">
   <inertial>
-    <origin xyz="0.0 0.03749999999999998 1.3877787807814457e-17" rpy="0 0 0"/>
-    <mass value="2.153167642492919"/>
-    <inertia ixx="0.006279" iyy="0.010596" izz="0.006279" ixy="0.0" iyz="0.0" ixz="0.0"/>
-  </inertial>
-  <visual>
-    <origin xyz="-0.0 -0.25 -0.1" rpy="0 0 0"/>
-    <geometry>
-      <mesh filename="file://$(find factory_amr_description)/meshes/left_wheel_1.stl" scale="0.001 0.001 0.001"/>
-    </geometry>
-    <material name="black"/>
-  </visual>
-  <collision>
-    <origin xyz="-0.0 -0.25 -0.1" rpy="0 0 0"/>
-    <geometry>
-      <mesh filename="file://$(find factory_amr_description)/meshes/left_wheel_1.stl" scale="0.001 0.001 0.001"/>
-    </geometry>
-  </collision>
-</link>
-<gazebo reference="left_wheel">
-  <material>Gazebo/Black</material>
-</gazebo>
-<link name="luggage">
-  <inertial>
-    <origin xyz="0.2776968707983327 -0.2999999999999999 0.08670656285317513" rpy="0 0 0"/>
+    <origin xyz="0.2776968707983327 0.3000000000000001 0.08670656285317513" rpy="0 0 0"/>
     <mass value="128.17276920688812"/>
     <inertia ixx="9.105387" iyy="8.394601" izz="16.079343" ixy="0.0" iyz="-0.0" ixz="-0.544919"/>
   </inertial>
   <visual>
-    <origin xyz="0.325 -0.3 -0.525" rpy="0 0 0"/>
+    <origin xyz="0.325 0.3 -0.525" rpy="0 0 0"/>
     <geometry>
       <mesh filename="file://$(find factory_amr_description)/meshes/revolute_1.stl" scale="0.001 0.001 0.001"/>
     </geometry>
-    <material name="orange"/>
+    <material name="silver"/>
   </visual>
   <collision>
-    <origin xyz="0.325 -0.3 -0.525" rpy="0 0 0"/>
+    <origin xyz="0.325 0.3 -0.525" rpy="0 0 0"/>
     <geometry>
       <mesh filename="file://$(find factory_amr_description)/meshes/revolute_1.stl" scale="0.001 0.001 0.001"/>
@@ -93,8 +84,5 @@
   </collision>
 </link>
-<gazebo reference="luggage">
-  <material>Gazebo/Orange</material>
-</gazebo>
-<link name="laser_frame">
+<link name="lidar_1">
   <inertial>
     <origin xyz="-7.237528875152536e-18 -1.447505775030507e-17 0.010000000000000009" rpy="0 0 0"/>
@@ -107,5 +95,5 @@
       <mesh filename="file://$(find factory_amr_description)/meshes/lidar_1.stl" scale="0.001 0.001 0.001"/>
     </geometry>
-    <material name="blue"/>
+    <material name="silver"/>
   </visual>
   <collision>
@@ -116,5 +104,25 @@
   </collision>
 </link>
-<link name="imu">
+<link name="camera_1">
+  <inertial>
+    <origin xyz="0.010000000000000009 0.0 0.0" rpy="0 0 0"/>
+    <mass value="0.19729201864543888"/>
+    <inertia ixx="3.9e-05" iyy="2.6e-05" izz="2.6e-05" ixy="0.0" iyz="0.0" ixz="0.0"/>
+  </inertial>
+  <visual>
+    <origin xyz="-0.39 -0.0 -0.475" rpy="0 0 0"/>
+    <geometry>
+      <mesh filename="file://$(find factory_amr_description)/meshes/camera_1.stl" scale="0.001 0.001 0.001"/>
+    </geometry>
+    <material name="silver"/>
+  </visual>
+  <collision>
+    <origin xyz="-0.39 -0.0 -0.475" rpy="0 0 0"/>
+    <geometry>
+      <mesh filename="file://$(find factory_amr_description)/meshes/camera_1.stl" scale="0.001 0.001 0.001"/>
+    </geometry>
+  </collision>
+</link>
+<link name="imu_1">
   <inertial>
     <origin xyz="0.0 0.0 -0.0050000000000000044" rpy="0 0 0"/>
@@ -127,5 +135,5 @@
       <mesh filename="file://$(find factory_amr_description)/meshes/imu_1.stl" scale="0.001 0.001 0.001"/>
     </geometry>
-    <material name="red"/>
+    <material name="silver"/>
   </visual>
   <collision>
@@ -136,118 +144,37 @@
   </collision>
 </link>
-<gazebo reference="imu">
-  <material>Gazebo/Red</material>
-</gazebo>
-<link name="camera">
-  <inertial>
-    <origin xyz="0.010000000000000064 0.0 0.0" rpy="0 0 0"/>
-    <mass value="0.19729201864543888"/>
-    <inertia ixx="3.9e-05" iyy="2.6e-05" izz="2.6e-05" ixy="0.0" iyz="-0.0" ixz="0.0"/>
-  </inertial>
-  <visual>
-    <origin xyz="-0.39 -0.0 -0.475" rpy="0 0 0"/>
-    <geometry>
-      <mesh filename="file://$(find factory_amr_description)/meshes/camera_1.stl" scale="0.001 0.001 0.001"/>
-    </geometry>
-    <material name="red"/>
-  </visual>
-  <collision>
-    <origin xyz="-0.39 -0.0 -0.475" rpy="0 0 0"/>
-    <geometry>
-      <mesh filename="file://$(find factory_amr_description)/meshes/camera_1.stl" scale="0.001 0.001 0.001"/>
-    </geometry>
-  </collision>
-</link>
-<joint name="right_wheel_joint" type="continuous">
+<joint name="Revolute 13" type="continuous">
+  <origin xyz="0.0 0.25 0.1" rpy="0 0 0"/>
+  <parent link="base_link"/>
+  <child link="left_wheel_1"/>
+  <axis xyz="0.0 1.0 0.0"/>
+</joint>
+<joint name="Revolute 14" type="continuous">
   <origin xyz="0.0 -0.25 0.1" rpy="0 0 0"/>
   <parent link="base_link"/>
-  <child link="right_wheel"/>
+  <child link="right_wheel_1"/>
   <axis xyz="0.0 -1.0 0.0"/>
 </joint>
-<joint name="left_wheel_joint" type="continuous">
-  <origin xyz="0.0 0.25 0.1" rpy="0 0 0"/>
+<joint name="Revolute 15" type="revolute">
+  <origin xyz="-0.325 -0.3 0.525" rpy="0 0 0"/>
   <parent link="base_link"/>
-  <child link="left_wheel"/>
-  <axis xyz="0.0 1.0 0.0"/>
-</joint>
-<joint name="luggage_joint" type="revolute">
-  <origin xyz="-0.325 0.3 0.525" rpy="0 0 0"/>
-  <parent link="base_link"/>
-  <child link="luggage"/>
+  <child link="revolute_1"/>
   <axis xyz="0.0 -1.0 0.0"/>
   <limit upper="0.785398" lower="0.0" effort="100" velocity="100"/>
 </joint>
-<joint name="laser_joint" type="fixed">
+<joint name="Rigid 16" type="fixed">
   <origin xyz="0.0 0.0 0.26" rpy="0 0 0"/>
   <parent link="base_link"/>
-  <child link="laser_frame"/>
+  <child link="lidar_1"/>
 </joint>
-<joint name="imu_joint" type="fixed">
+<joint name="Rigid 17" type="fixed">
+  <origin xyz="0.39 0.0 0.475" rpy="0 0 0"/>
+  <parent link="base_link"/>
+  <child link="camera_1"/>
+</joint>
+<joint name="Rigid 18" type="fixed">
   <origin xyz="0.0 0.0 0.23" rpy="0 0 0"/>
   <parent link="base_link"/>
-  <child link="imu"/>
+  <child link="imu_1"/>
 </joint>
-<joint name="camera_joint" type="fixed">
-  <origin xyz="0.39 0.0 0.475" rpy="0 0 0"/>
-  <parent link="base_link"/>
-  <child link="camera"/>
-</joint>
-<joint name="camera_optical_joint" type="fixed">
-  <origin xyz="0.0 0.0 0.0" rpy="${-pi/2} 0 ${-pi/2}"/>
-  <parent link="camera"/>
-  <child link="camera_optical"/>
-</joint>
-<link name="camera_optical" type="fixed"></link>
-<gazebo reference="laser_frame">
-  <material>Gazebo/Blue</material>
-  <sensor name="laser" type="ray">
-    <pose> 0 0 0 0 0 0 </pose>
-    <visualize>true</visualize>
-    <update_rate>10</update_rate>
-    <ray>
-      <scan>
-        <horizontal>
-          <samples>360</samples>
-          <resolution>1</resolution>
-          <min_angle>-3.14</min_angle>
-          <max_angle>3.14</max_angle>
-        </horizontal>
-      </scan>
-      <range>
-        <min>0.4</min>
-        <max>12</max>
-      </range>
-    </ray>
-    <plugin name="laser_controller" filename="libgazebo_ros_ray_sensor.so">
-      <ros>
-        <argument>~/out:=scan</argument>
-      </ros>
-      <output_type>sensor_msgs/LaserScan</output_type>
-      <frame_name>laser_frame</frame_name>
-    </plugin>
-  </sensor>
-</gazebo>
-<gazebo reference="camera">
-  <material>Gazebo/Red</material>
-  <sensor name="camera" type="camera">
-    <pose> 0 0 0 0 0 0 </pose>
-    <visualize>true</visualize>
-    <update_rate>10</update_rate>
-    <camera>
-      <horizontal_fov>1.089</horizontal_fov>
-      <image>
-        <format>R8G8B8</format>
-        <width>640</width>
-        <height>480</height>
-      </image>
-      <clip>
-        <near>0.05</near>
-        <far>8.0</far>
-      </clip>
-    </camera>
-    <plugin name="camera_controller" filename="libgazebo_ros_camera.so">
-      <frame_name>camera_optical</frame_name>
-    </plugin>
-  </sensor>
-</gazebo>
 </robot>

File: factory_amr_description/urdf/materials.xacro (robot description, xacro)
@@ -4,15 +4,3 @@
   <color rgba="0.700 0.700 0.700 1.000"/>
 </material>
-<material name="black">
-  <color rgba="0.000 0.000 0.000 1.000"/>
-</material>
-<material name="red">
-  <color rgba="0.800 0.000 0.000 1.000"/>
-</material>
-<material name="blue">
-  <color rgba="0.000 0.000 0.700 1.000"/>
-</material>
-<material name="orange">
-  <color rgba="1.000 0.4235 0.0392 1.000"/>
-</material>
 </robot>
