Commit message: Add Sensors
Add  LiDAR and Camera on robot

File: factory_amr_description/urdf/factory_amr.xacro (robot description, xacro)
@@ -1,180 +1,310 @@
 <?xml version="1.0" ?>
-<robot name="factory_amr" xmlns:xacro="http://www.ros.org/wiki/xacro">
-<xacro:include filename="$(find factory_amr_description)/urdf/materials.xacro" />
-<xacro:include filename="$(find factory_amr_description)/urdf/factory_amr.trans" />
-<xacro:include filename="$(find factory_amr_description)/urdf/factory_amr.gazebo" />
-<link name="base_link">
-  <inertial>
-    <origin xyz="-0.002396599951463409 2.104073385822183e-15 0.2688636212913025" rpy="0 0 0"/>
-    <mass value="29.324129559371645"/>
-    <inertia ixx="2.322166" iyy="2.720165" izz="3.470128" ixy="0.0" iyz="0.0" ixz="-0.006447"/>
-  </inertial>
-  <visual>
-    <origin xyz="0 0 0" rpy="0 0 0"/>
-    <geometry>
-      <mesh filename="file://$(find factory_amr_description)/meshes/base_link.stl" scale="0.001 0.001 0.001"/>
-    </geometry>
-    <material name="silver"/>
-  </visual>
-  <collision>
-    <origin xyz="0 0 0" rpy="0 0 0"/>
-    <geometry>
-      <mesh filename="file://$(find factory_amr_description)/meshes/base_link.stl" scale="0.001 0.001 0.001"/>
-    </geometry>
-  </collision>
-</link>
-<link name="left_wheel_1">
-  <inertial>
-    <origin xyz="0.0 0.03749999999999998 0.0" rpy="0 0 0"/>
-    <mass value="18.49612674800992"/>
-    <inertia ixx="0.05491" iyy="0.092481" izz="0.05491" ixy="0.0" iyz="0.0" ixz="0.0"/>
-  </inertial>
-  <visual>
-    <origin xyz="-0.0 -0.25 -0.1" rpy="0 0 0"/>
-    <geometry>
-      <mesh filename="file://$(find factory_amr_description)/meshes/left_wheel_1.stl" scale="0.001 0.001 0.001"/>
-    </geometry>
-    <material name="silver"/>
-  </visual>
-  <collision>
-    <origin xyz="-0.0 -0.25 -0.1" rpy="0 0 0"/>
-    <geometry>
-      <mesh filename="file://$(find factory_amr_description)/meshes/left_wheel_1.stl" scale="0.001 0.001 0.001"/>
-    </geometry>
-  </collision>
-</link>
-<link name="right_wheel_1">
-  <inertial>
-    <origin xyz="1.5440061600325417e-17 -0.03749999999999998 0.0" rpy="0 0 0"/>
-    <mass value="18.496126748009903"/>
-    <inertia ixx="0.05491" iyy="0.092481" izz="0.05491" ixy="-0.0" iyz="0.0" ixz="0.0"/>
-  </inertial>
-  <visual>
-    <origin xyz="-0.0 0.25 -0.1" rpy="0 0 0"/>
-    <geometry>
-      <mesh filename="file://$(find factory_amr_description)/meshes/right_wheel_1.stl" scale="0.001 0.001 0.001"/>
-    </geometry>
-    <material name="silver"/>
-  </visual>
-  <collision>
-    <origin xyz="-0.0 0.25 -0.1" rpy="0 0 0"/>
-    <geometry>
-      <mesh filename="file://$(find factory_amr_description)/meshes/right_wheel_1.stl" scale="0.001 0.001 0.001"/>
-    </geometry>
-  </collision>
-</link>
-<link name="revolute_1">
-  <inertial>
-    <origin xyz="0.2776968707983327 0.3000000000000001 0.08670656285317513" rpy="0 0 0"/>
-    <mass value="128.17276920688812"/>
-    <inertia ixx="9.105387" iyy="8.394601" izz="16.079343" ixy="0.0" iyz="-0.0" ixz="-0.544919"/>
-  </inertial>
-  <visual>
-    <origin xyz="0.325 0.3 -0.525" rpy="0 0 0"/>
-    <geometry>
-      <mesh filename="file://$(find factory_amr_description)/meshes/revolute_1.stl" scale="0.001 0.001 0.001"/>
-    </geometry>
-    <material name="silver"/>
-  </visual>
-  <collision>
-    <origin xyz="0.325 0.3 -0.525" rpy="0 0 0"/>
-    <geometry>
-      <mesh filename="file://$(find factory_amr_description)/meshes/revolute_1.stl" scale="0.001 0.001 0.001"/>
-    </geometry>
-  </collision>
-</link>
-<link name="lidar_1">
-  <inertial>
-    <origin xyz="-7.237528875152536e-18 -1.447505775030507e-17 0.010000000000000009" rpy="0 0 0"/>
-    <mass value="1.2330751165339937"/>
-    <inertia ixx="0.000812" iyy="0.000812" izz="0.001541" ixy="-0.0" iyz="0.0" ixz="0.0"/>
-  </inertial>
-  <visual>
-    <origin xyz="-0.0 -0.0 -0.26" rpy="0 0 0"/>
-    <geometry>
-      <mesh filename="file://$(find factory_amr_description)/meshes/lidar_1.stl" scale="0.001 0.001 0.001"/>
-    </geometry>
-    <material name="silver"/>
-  </visual>
-  <collision>
-    <origin xyz="-0.0 -0.0 -0.26" rpy="0 0 0"/>
-    <geometry>
-      <mesh filename="file://$(find factory_amr_description)/meshes/lidar_1.stl" scale="0.001 0.001 0.001"/>
-    </geometry>
-  </collision>
-</link>
-<link name="camera_1">
-  <inertial>
-    <origin xyz="0.010000000000000009 0.0 0.0" rpy="0 0 0"/>
-    <mass value="0.19729201864543888"/>
-    <inertia ixx="3.9e-05" iyy="2.6e-05" izz="2.6e-05" ixy="0.0" iyz="0.0" ixz="0.0"/>
-  </inertial>
-  <visual>
-    <origin xyz="-0.39 -0.0 -0.475" rpy="0 0 0"/>
-    <geometry>
-      <mesh filename="file://$(find factory_amr_description)/meshes/camera_1.stl" scale="0.001 0.001 0.001"/>
-    </geometry>
-    <material name="silver"/>
-  </visual>
-  <collision>
-    <origin xyz="-0.39 -0.0 -0.475" rpy="0 0 0"/>
-    <geometry>
-      <mesh filename="file://$(find factory_amr_description)/meshes/camera_1.stl" scale="0.001 0.001 0.001"/>
-    </geometry>
-  </collision>
-</link>
-<link name="imu_1">
-  <inertial>
-    <origin xyz="0.0 0.0 -0.0050000000000000044" rpy="0 0 0"/>
-    <mass value="0.1256"/>
-    <inertia ixx="1.8e-05" iyy="1.8e-05" izz="3.3e-05" ixy="0.0" iyz="0.0" ixz="0.0"/>
-  </inertial>
-  <visual>
-    <origin xyz="-0.0 -0.0 -0.23" rpy="0 0 0"/>
-    <geometry>
-      <mesh filename="file://$(find factory_amr_description)/meshes/imu_1.stl" scale="0.001 0.001 0.001"/>
-    </geometry>
-    <material name="silver"/>
-  </visual>
-  <collision>
-    <origin xyz="-0.0 -0.0 -0.23" rpy="0 0 0"/>
-    <geometry>
-      <mesh filename="file://$(find factory_amr_description)/meshes/imu_1.stl" scale="0.001 0.001 0.001"/>
-    </geometry>
-  </collision>
-</link>
-<joint name="Revolute 13" type="continuous">
-  <origin xyz="0.0 0.25 0.1" rpy="0 0 0"/>
-  <parent link="base_link"/>
-  <child link="left_wheel_1"/>
-  <axis xyz="0.0 1.0 0.0"/>
-</joint>
-<joint name="Revolute 14" type="continuous">
-  <origin xyz="0.0 -0.25 0.1" rpy="0 0 0"/>
-  <parent link="base_link"/>
-  <child link="right_wheel_1"/>
-  <axis xyz="0.0 -1.0 0.0"/>
-</joint>
-<joint name="Revolute 15" type="revolute">
-  <origin xyz="-0.325 -0.3 0.525" rpy="0 0 0"/>
-  <parent link="base_link"/>
-  <child link="revolute_1"/>
-  <axis xyz="0.0 -1.0 0.0"/>
-  <limit upper="0.785398" lower="0.0" effort="100" velocity="100"/>
-</joint>
-<joint name="Rigid 16" type="fixed">
-  <origin xyz="0.0 0.0 0.26" rpy="0 0 0"/>
-  <parent link="base_link"/>
-  <child link="lidar_1"/>
-</joint>
-<joint name="Rigid 17" type="fixed">
-  <origin xyz="0.39 0.0 0.475" rpy="0 0 0"/>
-  <parent link="base_link"/>
-  <child link="camera_1"/>
-</joint>
-<joint name="Rigid 18" type="fixed">
-  <origin xyz="0.0 0.0 0.23" rpy="0 0 0"/>
-  <parent link="base_link"/>
-  <child link="imu_1"/>
-</joint>
+<robot xmlns:xacro="http://www.ros.org/wiki/xacro">
+  <xacro:include filename="inertial_macros.xacro"/>
+  <xacro:include filename="$(find factory_amr_description)/urdf/materials.xacro" />
+  <xacro:include filename="$(find factory_amr_description)/urdf/factory_amr.trans" />
+  <xacro:include filename="$(find factory_amr_description)/urdf/factory_amr.gazebo" />
+  <link name="base_link">
+    <inertial>
+      <origin xyz="-0.002396599951463409 2.104073385822183e-15 0.2688636212913025" rpy="0 0 0"/>
+      <mass value="29.324129559371645"/>
+      <inertia ixx="2.322166" iyy="2.720165" izz="3.470128" ixy="0.0" iyz="0.0" ixz="-0.006447"/>
+    </inertial>
+    <visual>
+      <origin xyz="0 0 0" rpy="0 0 0"/>
+      <geometry>
+        <mesh filename="file://$(find factory_amr_description)/meshes/base_link.stl" scale="0.001 0.001 0.001"/>
+      </geometry>
+      <material name="silver"/>
+    </visual>
+    <collision>
+      <origin xyz="0 0 0" rpy="0 0 0"/>
+      <geometry>
+        <mesh filename="file://$(find factory_amr_description)/meshes/base_link.stl" scale="0.001 0.001 0.001"/>
+      </geometry>
+    </collision>
+  </link>
+  <gazebo reference="base_link">
+    <material>Gazebo/White</material>
+  </gazebo>
+  <link name="right_wheel_link">
+    <inertial>
+      <origin xyz="-1.5713222806367798e-17 -0.03750000000000003 0.0" rpy="0 0 0"/>
+      <mass value="2.1531676424929196"/>
+      <inertia ixx="0.006279" iyy="0.010596" izz="0.006279" ixy="0.0" iyz="-0.0" ixz="-0.0"/>
+    </inertial>
+    <visual>
+      <origin xyz="-0.0 -0.1 -0.25" rpy="-${pi/2} 0 0"/>
+      <geometry>
+        <mesh filename="file://$(find factory_amr_description)/meshes/right_wheel_1.stl" scale="0.001 0.001 0.001" rpy="0 0 0"/>
+      </geometry>
+      <material name="black"/>
+    </visual>
+    <collision>
+      <origin xyz="-0.0 -0.1 -0.25" rpy="-${pi/2} 0 0"/>
+      <geometry>
+        <mesh filename="file://$(find factory_amr_description)/meshes/right_wheel_1.stl" scale="0.001 0.001 0.001"/>
+      </geometry>
+    </collision>
+  </link>
+  <gazebo reference="right_wheel_link">
+    <material>Gazebo/Black</material>
+  </gazebo>
+  <link name="left_wheel_link">
+    <inertial>
+      <origin xyz="0.0 0.03749999999999998 1.3877787807814457e-17" rpy="0 0 0"/>
+      <mass value="2.153167642492919"/>
+      <inertia ixx="0.006279" iyy="0.010596" izz="0.006279" ixy="0.0" iyz="0.0" ixz="0.0"/>
+    </inertial>
+    <visual>
+      <origin xyz="0 0.1 -0.25" rpy="${pi/2} 0 0"/>
+      <geometry>
+        <mesh filename="file://$(find factory_amr_description)/meshes/left_wheel_1.stl" scale="0.001 0.001 0.001" rpy="0 0 0"/>
+      </geometry>
+      <material name="black"/>
+    </visual>
+    <collision>
+      <origin xyz="0 0.1 -0.25" rpy="${pi/2} 0 0"/>
+      <geometry>
+        <mesh filename="file://$(find factory_amr_description)/meshes/left_wheel_1.stl" scale="0.001 0.001 0.001"/>
+      </geometry>
+    </collision>
+  </link>
+  <gazebo reference="left_wheel_link">
+    <material>Gazebo/Black</material>
+  </gazebo>
+  <link name="luggage_link">
+    <inertial>
+      <origin xyz="0.2776968707983327 -0.2999999999999999 0.08670656285317513" rpy="0 0 0"/>
+      <mass value="128.17276920688812"/>
+      <inertia ixx="9.105387" iyy="8.394601" izz="16.079343" ixy="0.0" iyz="-0.0" ixz="-0.544919"/>
+    </inertial>
+    <visual>
+      <origin xyz="0.325 -0.3 -0.525" rpy="0 0 0"/>
+      <geometry>
+        <mesh filename="file://$(find factory_amr_description)/meshes/revolute_1.stl" scale="0.001 0.001 0.001"/>
+      </geometry>
+      <material name="orange"/>
+    </visual>
+    <collision>
+      <origin xyz="0.325 -0.3 -0.525" rpy="0 0 0"/>
+      <geometry>
+        <mesh filename="file://$(find factory_amr_description)/meshes/revolute_1.stl" scale="0.001 0.001 0.001"/>
+      </geometry>
+    </collision>
+  </link>
+  <gazebo reference="luggage_link">
+    <material>Gazebo/Orange</material>
+  </gazebo>
+  <link name="imu_link">
+    <inertial>
+      <origin xyz="0.0 0.0 -0.0050000000000000044" rpy="0 0 0"/>
+      <mass value="0.1256"/>
+      <inertia ixx="1.8e-05" iyy="1.8e-05" izz="3.3e-05" ixy="0.0" iyz="0.0" ixz="0.0"/>
+    </inertial>
+    <visual>
+      <origin xyz="-0.0 -0.0 -0.23" rpy="0 0 0"/>
+      <geometry>
+        <mesh filename="file://$(find factory_amr_description)/meshes/imu_1.stl" scale="0.001 0.001 0.001"/>
+      </geometry>
+      <material name="red"/>
+    </visual>
+    <collision>
+      <origin xyz="-0.0 -0.0 -0.23" rpy="0 0 0"/>
+      <geometry>
+        <mesh filename="file://$(find factory_amr_description)/meshes/imu_1.stl" scale="0.001 0.001 0.001"/>
+      </geometry>
+    </collision>
+  </link>
+  <gazebo reference="imu_link">
+    <material>Gazebo/Red</material>
+  </gazebo>
+  <link name="camera_link">
+    <inertial>
+      <origin xyz="0.010000000000000064 0.0 0.0" rpy="0 0 0"/>
+      <mass value="0.19729201864543888"/>
+      <inertia ixx="3.9e-05" iyy="2.6e-05" izz="2.6e-05" ixy="0.0" iyz="-0.0" ixz="0.0"/>
+    </inertial>
+    <visual>
+      <origin xyz="-0.39 -0.0 -0.475" rpy="0 0 0"/>
+      <geometry>
+        <mesh filename="file://$(find factory_amr_description)/meshes/camera_1.stl" scale="0.001 0.001 0.001"/>
+      </geometry>
+      <material name="red"/>
+    </visual>
+    <collision>
+      <origin xyz="-0.39 -0.0 -0.475" rpy="0 0 0"/>
+      <geometry>
+        <mesh filename="file://$(find factory_amr_description)/meshes/camera_1.stl" scale="0.001 0.001 0.001"/>
+      </geometry>
+    </collision>
+  </link>
+  <!-- caster wheels -->
+  <joint name="front_caster" type="fixed">
+    <parent link="base_link"/>
+    <child link="front_caster_link"/>
+    <origin xyz="0.3 0 0.05"/>
+  </joint>
+  <link name="front_caster_link">
+    <visual>
+      <geometry>
+        <sphere radius="0.05"/>
+      </geometry>
+      <material name="black"/>
+    </visual>
+    <collision>
+      <geometry>
+        <sphere radius="0.05"/>
+      </geometry>
+    </collision>
+    <xacro:inertial_sphere mass="0.1" radius="0.05">
+      <origin xyz="0 0 0" rpy="0 0 0"/>
+    </xacro:inertial_sphere>
+  </link>
+  <gazebo reference="front_caster">
+    <material>Gazebo/Black</material>
+    <mu1 value="0.001"/>
+    <mu2 value="0.001"/>
+  </gazebo>
+  <joint name="back_caster" type="fixed">
+    <parent link="base_link"/>
+    <child link="back_caster_link"/>
+    <origin xyz="-0.3 0 0.05"/>
+  </joint>
+  <link name="back_caster_link">
+    <visual>
+      <geometry>
+        <sphere radius="0.05"/>
+      </geometry>
+      <material name="black"/>
+    </visual>
+    <collision>
+      <geometry>
+        <sphere radius="0.05"/>
+      </geometry>
+    </collision>
+    <xacro:inertial_sphere mass="0.1" radius="0.05">
+      <origin xyz="0 0 0" rpy="0 0 0"/>
+    </xacro:inertial_sphere>
+  </link>
+  <gazebo reference="back_caster">
+    <material>Gazebo/Black</material>
+    <mu1 value="0.001"/>
+    <mu2 value="0.001"/>
+  </gazebo>
+  <!-- joints -->
+  <joint name="right_wheel_joint" type="continuous">
+    <origin xyz="0.0 -0.25 0.1" rpy="${pi/2} 0 0"/>
+    <parent link="base_link"/>
+    <child link="right_wheel_link"/>
+    <axis xyz="0.0 0.0 -1.0"/>
+  </joint>
+  <joint name="left_wheel_joint" type="continuous">
+    <origin xyz="0.0 0.25 0.1" rpy="-${pi/2} 0 0"/>
+    <parent link="base_link"/>
+    <child link="left_wheel_link"/>
+    <axis xyz="0.0 0.0 1.0"/>
+  </joint>
+  <joint name="luggage_joint" type="revolute">
+    <origin xyz="-0.325 0.3 0.525" rpy="0 0 0"/>
+    <parent link="base_link"/>
+    <child link="luggage_link"/>
+    <axis xyz="0.0 -1.0 0.0"/>
+    <limit upper="0.785398" lower="0.0" effort="100" velocity="100"/>
+  </joint>
+  <joint name="imu_joint" type="fixed">
+    <origin xyz="0.0 0.0 0.23" rpy="0 0 0"/>
+    <parent link="base_link"/>
+    <child link="imu_link"/>
+  </joint>
+  <joint name="camera_joint" type="fixed">
+    <origin xyz="0.39 0.0 0.475" rpy="0 0 0"/>
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
File: factory_amr_description/urdf/materials.xacro (robot description, xacro)
@@ -4,3 +4,15 @@
   <color rgba="0.700 0.700 0.700 1.000"/>
 </material>
+<material name="black">
+  <color rgba="0.000 0.000 0.000 1.000"/>
+</material>
+<material name="red">
+  <color rgba="0.800 0.000 0.000 1.000"/>
+</material>
+<material name="blue">
+  <color rgba="0.000 0.000 0.700 1.000"/>
+</material>
+<material name="orange">
+  <color rgba="1.000 0.4235 0.0392 1.000"/>
+</material>
 </robot>

Commit message: modify some parameters

File: factory_amr_description/urdf/factory_amr.xacro (robot description, xacro)
@@ -8,5 +8,5 @@
     <inertial>
       <origin xyz="-0.002396599951463409 2.104073385822183e-15 0.2688636212913025" rpy="0 0 0"/>
-      <mass value="29.324129559371645"/>
+      <mass value="5"/>
       <inertia ixx="2.322166" iyy="2.720165" izz="3.470128" ixy="0.0" iyz="0.0" ixz="-0.006447"/>
     </inertial>
@@ -31,9 +31,9 @@
     <inertial>
       <origin xyz="-1.5713222806367798e-17 -0.03750000000000003 0.0" rpy="0 0 0"/>
-      <mass value="2.1531676424929196"/>
+      <mass value="0.5"/>
       <inertia ixx="0.006279" iyy="0.010596" izz="0.006279" ixy="0.0" iyz="-0.0" ixz="-0.0"/>
     </inertial>
     <visual>
-      <origin xyz="-0.0 -0.1 -0.25" rpy="-${pi/2} 0 0"/>
+      <origin xyz="-0.0 -0.1 -0.24" rpy="-${pi/2} 0 0"/>
       <geometry>
         <mesh filename="file://$(find factory_amr_description)/meshes/right_wheel_1.stl" scale="0.001 0.001 0.001" rpy="0 0 0"/>
@@ -42,5 +42,5 @@
     </visual>
     <collision>
-      <origin xyz="-0.0 -0.1 -0.25" rpy="-${pi/2} 0 0"/>
+      <origin xyz="-0.0 -0.1 -0.24" rpy="-${pi/2} 0 0"/>
       <geometry>
         <mesh filename="file://$(find factory_amr_description)/meshes/right_wheel_1.stl" scale="0.001 0.001 0.001"/>
@@ -54,9 +54,9 @@
     <inertial>
       <origin xyz="0.0 0.03749999999999998 1.3877787807814457e-17" rpy="0 0 0"/>
-      <mass value="2.153167642492919"/>
+      <mass value="0.5"/>
       <inertia ixx="0.006279" iyy="0.010596" izz="0.006279" ixy="0.0" iyz="0.0" ixz="0.0"/>
     </inertial>
     <visual>
-      <origin xyz="0 0.1 -0.25" rpy="${pi/2} 0 0"/>
+      <origin xyz="0 0.1 -0.24" rpy="${pi/2} 0 0"/>
       <geometry>
         <mesh filename="file://$(find factory_amr_description)/meshes/left_wheel_1.stl" scale="0.001 0.001 0.001" rpy="0 0 0"/>
@@ -65,5 +65,5 @@
     </visual>
     <collision>
-      <origin xyz="0 0.1 -0.25" rpy="${pi/2} 0 0"/>
+      <origin xyz="0 0.1 -0.24" rpy="${pi/2} 0 0"/>
       <geometry>
         <mesh filename="file://$(find factory_amr_description)/meshes/left_wheel_1.stl" scale="0.001 0.001 0.001"/>
@@ -77,5 +77,5 @@
     <inertial>
       <origin xyz="0.2776968707983327 -0.2999999999999999 0.08670656285317513" rpy="0 0 0"/>
-      <mass value="128.17276920688812"/>
+      <mass value="3"/>
       <inertia ixx="9.105387" iyy="8.394601" izz="16.079343" ixy="0.0" iyz="-0.0" ixz="-0.544919"/>
     </inertial>

File: factory_amr_description/urdf/gazebo_control.xacro (robot description, xacro)
@@ -5,8 +5,8 @@
             <left_joint>left_wheel_joint</left_joint>
             <right_joint>right_wheel_joint</right_joint>
-            <wheel_separation>0.6</wheel_separation>
+            <wheel_separation>0.62</wheel_separation>
             <wheel_diameter>1.0</wheel_diameter>
-            <max_wheel_torque>200</max_wheel_torque>
-            <max_wheel_acceleration>10.0</max_wheel_acceleration>
+            <max_wheel_torque>300</max_wheel_torque>
+            <max_wheel_acceleration>30.0</max_wheel_acceleration>
             <odometry_frame>odom</odometry_frame>
             <robot_base_frame>base_link</robot_base_frame>
